Commit message: added prefix support for gripper

File: src/kuka_lbr_iisy_support/urdf/gripper.urdf.xacro (robot description, xacro)
@@ -1,5 +1,6 @@
 <?xml version="1.0" encoding="UTF-8"?>
-<robot xmlns:xacro="http://wiki.ros.org/xacro" name="robotiq_gripper">
-    <link name="robotiq_85_base_link">
+<robot xmlns:xacro="http://wiki.ros.org/xacro">
+  <xacro:macro name="robotiq_gripper" params="prefix">
+    <link name="${prefix}robotiq_85_base_link">
       <visual>
         <geometry>
@@ -20,20 +21,20 @@
       </inertial>
     </link>
-    <joint name="robotiq_85_left_knuckle_joint" type="revolute">
-      <parent link="robotiq_85_base_link"/>
-      <child link="robotiq_85_left_knuckle_link"/>
+    <joint name="${prefix}robotiq_85_left_knuckle_joint" type="revolute">
+      <parent link="${prefix}robotiq_85_base_link"/>
+      <child link="${prefix}robotiq_85_left_knuckle_link"/>
       <axis xyz="0 0 1"/>
       <origin rpy="3.14 0.0 0.0" xyz="0.05490451627 0.03060114443 0.0"/>
       <limit lower="0.0" upper="0.80285" velocity="3.14" effort="1000"/>
     </joint>
-    <joint name="robotiq_85_right_knuckle_joint" type="revolute">
-      <parent link="robotiq_85_base_link"/>
-      <child link="robotiq_85_right_knuckle_link"/>
+    <joint name="${prefix}robotiq_85_right_knuckle_joint" type="revolute">
+      <parent link="${prefix}robotiq_85_base_link"/>
+      <child link="${prefix}robotiq_85_right_knuckle_link"/>
       <axis xyz="0 0 1"/>
       <origin rpy="0.0 0.0 0.0" xyz="0.05490451627 -0.03060114443 0.0"/>
       <limit lower="-3.14" upper="3.14" velocity="3.14" effort="1000"/>
-      <mimic joint="robotiq_85_left_knuckle_joint"/>
-    </joint>
-    <link name="robotiq_85_left_knuckle_link">
+      <mimic joint="${prefix}robotiq_85_left_knuckle_joint"/>
+    </joint>
+    <link name="${prefix}robotiq_85_left_knuckle_link">
       <visual>
         <geometry>
@@ -54,5 +55,5 @@
       </inertial>
     </link>
-    <link name="robotiq_85_right_knuckle_link">
+    <link name="${prefix}robotiq_85_right_knuckle_link">
       <visual>
         <geometry>
@@ -73,15 +74,15 @@
       </inertial>
     </link>
-    <joint name="robotiq_85_left_finger_joint" type="fixed">
-      <parent link="robotiq_85_left_knuckle_link"/>
-      <child link="robotiq_85_left_finger_link"/>
+    <joint name="${prefix}robotiq_85_left_finger_joint" type="fixed">
+      <parent link="${prefix}robotiq_85_left_knuckle_link"/>
+      <child link="${prefix}robotiq_85_left_finger_link"/>
       <origin xyz="-0.00408552455 -0.03148604435 0.0" rpy="0 0 0" />
     </joint>
-    <joint name="robotiq_85_right_finger_joint" type="fixed">
-      <parent link="robotiq_85_right_knuckle_link"/>
-      <child link="robotiq_85_right_finger_link"/>
+    <joint name="${prefix}robotiq_85_right_finger_joint" type="fixed">
+      <parent link="${prefix}robotiq_85_right_knuckle_link"/>
+      <child link="${prefix}robotiq_85_right_finger_link"/>
       <origin xyz="-0.00408552455 -0.03148604435 0.0" rpy="0 0 0" />
     </joint>
-    <link name="robotiq_85_left_finger_link">
+    <link name="${prefix}robotiq_85_left_finger_link">
       <visual>
         <geometry>
@@ -102,5 +103,5 @@
       </inertial>
     </link>
-    <link name="robotiq_85_right_finger_link">
+    <link name="${prefix}robotiq_85_right_finger_link">
       <visual>
         <geometry>
@@ -121,21 +122,21 @@
       </inertial>
     </link>
-    <joint name="robotiq_85_left_inner_knuckle_joint" type="revolute">
-      <parent link="robotiq_85_base_link"/>
-      <child link="robotiq_85_left_inner_knuckle_link"/>
+    <joint name="${prefix}robotiq_85_left_inner_knuckle_joint" type="revolute">
+      <parent link="${prefix}robotiq_85_base_link"/>
+      <child link="${prefix}robotiq_85_left_inner_knuckle_link"/>
       <axis xyz="0 0 1"/>
       <origin xyz="0.06142 0.0127 0" rpy="3.14 0.0 0.0" />
       <limit lower="-3.14" upper="3.14" velocity="3.14" effort="0.1"/>
-      <mimic joint="robotiq_85_left_knuckle_joint" offset="0"/>
-    </joint>
-    <joint name="robotiq_85_right_inner_knuckle_joint" type="revolute">
-      <parent link="robotiq_85_base_link"/>
-      <child link="robotiq_85_right_inner_knuckle_link"/>
+      <mimic joint="${prefix}robotiq_85_left_knuckle_joint" offset="0"/>
+    </joint>
+    <joint name="${prefix}robotiq_85_right_inner_knuckle_joint" type="revolute">
+      <parent link="${prefix}robotiq_85_base_link"/>
+      <child link="${prefix}robotiq_85_right_inner_knuckle_link"/>
       <axis xyz="0 0 1"/>
       <origin xyz="0.06142 -0.0127 0" rpy="0 0 0"/>
       <limit lower="-3.14" upper="3.14" velocity="3.14" effort="0.1"/>
-      <mimic joint="robotiq_85_left_knuckle_joint" offset="0"/>
-    </joint>
-    <link name="robotiq_85_left_inner_knuckle_link">
+      <mimic joint="${prefix}robotiq_85_left_knuckle_joint" offset="0"/>
+    </joint>
+    <link name="${prefix}robotiq_85_left_inner_knuckle_link">
       <visual>
         <geometry>
@@ -156,5 +157,5 @@
       </inertial>
     </link>
-    <link name="robotiq_85_right_inner_knuckle_link">
+    <link name="${prefix}robotiq_85_right_inner_knuckle_link">
       <visual>
         <geometry>
@@ -175,21 +176,21 @@
       </inertial>
     </link>
-    <joint name="robotiq_85_left_finger_tip_joint" type="revolute">
-      <parent link="robotiq_85_left_inner_knuckle_link"/>
-      <child link="robotiq_85_left_finger_tip_link"/>
+    <joint name="${prefix}robotiq_85_left_finger_tip_joint" type="revolute">
+      <parent link="${prefix}robotiq_85_left_inner_knuckle_link"/>
+      <child link="${prefix}robotiq_85_left_finger_tip_link"/>
       <axis xyz="0 0 1"/>
       <origin xyz="0.04303959807 -0.03759940821 0.0" rpy="0.0 0.0 0.0"/>
       <limit lower="-3.14" upper="3.14" velocity="3.14" effort="0.1"/>
-      <mimic joint="robotiq_85_left_knuckle_joint" multiplier="-1"/>
-    </joint>
-    <joint name="robotiq_85_right_finger_tip_joint" type="revolute">
-      <parent link="robotiq_85_right_inner_knuckle_link"/>
-      <child link="robotiq_85_right_finger_tip_link"/>
+      <mimic joint="${prefix}robotiq_85_left_knuckle_joint" multiplier="-1"/>
+    </joint>
+    <joint name="${prefix}robotiq_85_right_finger_tip_joint" type="revolute">
+      <parent link="${prefix}robotiq_85_right_inner_knuckle_link"/>
+      <child link="${prefix}robotiq_85_right_finger_tip_link"/>
       <axis xyz="0 0 1"/>
       <origin rpy="0.0 0.0 0.0" xyz="0.04303959807 -0.03759940821  0.0"/>
       <limit lower="-3.14" upper="3.14" velocity="3.14" effort="0.1"/>
-      <mimic joint="robotiq_85_left_knuckle_joint" multiplier="-1"/>
-    </joint>
-    <link name="robotiq_85_left_finger_tip_link">
+      <mimic joint="${prefix}robotiq_85_left_knuckle_joint" multiplier="-1"/>
+    </joint>
+    <link name="${prefix}robotiq_85_left_finger_tip_link">
       <visual>
         <geometry>
@@ -210,5 +211,5 @@
       </inertial>
     </link>
-    <link name="robotiq_85_right_finger_tip_link">
+    <link name="${prefix}robotiq_85_right_finger_tip_link">
       <visual>
         <geometry>
@@ -229,3 +230,4 @@
       </inertial>
     </link>
+  </xacro:macro>
 </robot>

File: src/kuka_lbr_iisy_support/urdf/lbr_iisy3_r760.urdf.xacro (robot description, xacro)
@@ -5,4 +5,6 @@
   <!-- Read additional arguments  -->
   <xacro:arg name="prefix" default=""/>
+  <!-- Global world link -->
+  <link name="world"/>
   <xacro:arg name="x" default="0"/>
   <xacro:arg name="y" default="0"/>
