Commit message: added dual robot description

File: src/kuka_lbr_iisy_support/urdf/lbr_iisy3_r760_macro.xacro (robot description, xacro)
@@ -6,5 +6,5 @@
   <xacro:include filename="$(find kuka_lbr_iisy_support)/urdf/gripper.urdf.xacro"/>
   <xacro:macro name="kuka_lbr_iisy3_r760_robot" params="prefix *origin">
-    <link name="world"/>
+    <!-- <link name="world"/> -->
     <link name="${prefix}base_link">
       <collision>
@@ -181,6 +181,7 @@
       <parent link="${prefix}link_6"/>
     </joint>-->
-    <joint name="gripper_joint" type="fixed">
-      <child link="robotiq_85_base_link"/>
+    <xacro:robotiq_gripper prefix="${prefix}"/>
+    <joint name="${prefix}gripper_joint" type="fixed">
+      <child link="${prefix}robotiq_85_base_link"/>
       <origin rpy="0 0 0" xyz="0.0 0.0 0.0"/>
       <parent link="${prefix}flange"/>
